File: lcr/kicad/COG12864/lcr.sch (KiCad schematic (older format))
At the start: 98 parts, among them SW1 SW_Push, SW2 SW_Push, U1 N32G430C8L7, U2 LMV722, U3 LMV722, U4 LMV722, U5 LMV722, U6 LMV722, U7 74HC4053, U8 LMV722, Y1 8MHZ

Commit message: 添加阿拉伯数字字库
Parts:
- removed C14, C15, C16, C?: 106, symbol Device:C
- removed C? (x2): 104, symbol Device:C
- removed C? (x3): C, symbol Device:C
- removed Q? (x3): BC547, Package_TO_SOT_THT:TO-92_Inline, symbol Transistor_BJT:BC547
- removed R2: 100, symbol Device:R
- removed R3: 10K, symbol Device:R
- removed R? (x2): 100K, symbol Device:R
- removed R? (x2): R, symbol Device:R
- removed R? (x3): 1K, symbol Device:R
- removed U3: LMV722, symbol Analog_Switch:CD4053B
- removed U7: 74HC4053, symbol Analog_Switch:CD4053B
- added C? (x16): C, symbol Device:C
- added J?: Conn_01x03_Male, symbol Connector:Conn_01x03_Male
- added J?: Conn_01x04_Male, symbol Connector:Conn_01x04_Male
- added R?: 100K, symbol Device:R
- added R?: 10K, symbol Device:R
- added R?: 1K, symbol Device:R
- added R?: 100, symbol Device:R
- added R? (x9): R, symbol Device:R
- added U?: CD4052B, symbol Analog_Switch:CD4052B
- added U?: CD4053B, symbol Analog_Switch:CD4053B
- C? (x3): value 104 -> 106
- R? (x2): value 900 -> 9K
- R? (x3): value 100 -> 1K
- R?: value 100 -> 500
- R?: value 1K -> 500
Connections:
- net labels added: SIN
- net labels removed: PA3_100_10K_dangwei, PB10_100HZ_lvbo, PB1_10K_lvbo, PB2_1K_lvbo
- wire segments 378 -> 404
Other:
- moved on the sheet: C1, C13, C17, C18, C19, C2, C20, C21, C22, C3, C4, C5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
